Commit message: fix: changed some incorrect masses that was calculated using material density to real mass (hopefully), corrected URDF and MJCF files

File: resources/robots/Xuanwu/urdf/Xuanwu.urdf (robot description, URDF)
Before this commit: robot Xuanwu, 11 links, 10 joints
Links:
- link base_link: mass 1.894 -> 2.14
- link link_1: mass 0.547 -> 0.469
- link link_10: mass 0.105 -> 0.107
- link link_2: mass 0.378 -> 0.364
- link link_3: mass 0.436 -> 0.475
- link link_4: mass 0.436 -> 0.475
- link link_5: mass 0.105 -> 0.107
- link link_6: mass 0.547 -> 0.574
- link link_7: mass 0.378 -> 0.364
- link link_8: mass 0.436 -> 0.475
- link link_9: mass 0.436 -> 0.475

Commit message: feat: changed kp based on actual torque and simulation torque discrepancy analysis

File: resources/robots/Xuanwu/urdf/Xuanwu.urdf (robot description, URDF)
Before this commit: robot Xuanwu, 11 links, 10 joints
Links:
- link link_6: mass 0.574 -> 0.469

Commit message: feat: changed PD setting and URDF file

File: resources/robots/Xuanwu/urdf/Xuanwu.urdf (robot description, URDF)
Before this commit: robot Xuanwu, 11 links, 10 joints
Links:
- link base_link: mass 2.14 -> 1.42

Commit message: fix: fixed mass properties

File: resources/robots/Xuanwu/urdf/Xuanwu.urdf (robot description, URDF)
Before this commit: robot Xuanwu, 11 links, 10 joints
Links:
- link base_link: mass 1.42 -> 1.874

Commit message: fix: fixed URDF, MJCF, and meshes

File: resources/robots/Xuanwu/urdf/Xuanwu.urdf (robot description, URDF)
Before this commit: robot Xuanwu, 11 links, 10 joints
Links:
- link base_link: mass 1.874 -> 2.016243
- link link_1: mass 0.469 -> 0.504
- link link_10: mass 0.107 -> 0.122
- link link_2: mass 0.364 -> 0.390
- link link_3: mass 0.475 -> 0.481
- link link_4: mass 0.475 -> 0.481
- link link_5: mass 0.107 -> 0.122
- link link_6: mass 0.574 -> 0.504
- link link_7: mass 0.364 -> 0.390
- link link_8: mass 0.475 -> 0.481
- link link_9: mass 0.475 -> 0.481
Joints:
- joint joint_1: origin xyz=-0.073 0 -0.001 rpy=0 0 0 -> xyz=-0.073035 -1.4472E-05 -0.00095242 rpy=0 0 0
- joint joint_10: origin xyz=0 0 -0.18 rpy=0 0 0 -> xyz=-5E-05 1.1901E-05 -0.18002 rpy=0 0 0
- joint joint_2: origin xyz=0 -0.083 -0.11 rpy=0 0 0 -> xyz=4.9294E-05 -0.083183 -0.11003 rpy=0 0 0
- joint joint_3: origin xyz=0 0.082 0 rpy=0 0 0 -> xyz=0.00098795 0.082032 2.035E-05 rpy=0 0 0
- joint joint_4: origin xyz=0 0 -0.18 rpy=0 0 0 -> xyz=5E-05 -5.7742E-05 -0.17996 rpy=0 0 0
- joint joint_5: origin xyz=0 0 -0.18 rpy=0 0 0 -> xyz=5E-05 3.7392E-05 -0.18 rpy=0 0 0
- joint joint_6: origin xyz=0.073 0 -0.001 rpy=0 0 0 -> xyz=0.073035 1.4472E-05 -0.00095242 rpy=0 0 0
- joint joint_7: origin xyz=0 -0.083 -0.11 rpy=0 0 0 -> xyz=-2.035E-05 -0.083212 -0.11003 rpy=0 0 0
- joint joint_8: origin xyz=0 0.082 0 rpy=0 0 0 -> xyz=-0.0010169 0.082032 4.9294E-05 rpy=0 0 0
- joint joint_9: origin xyz=0 0 -0.18 rpy=0 0 0 -> xyz=-5E-05 -1.1901E-05 -0.17998 rpy=0 0 0
